File: PCB/CoolAwesomeHackpad.kicad_pcb (KiCad board)
At the start: 2 copper layers, 92 x 48 mm, 8 parts, among them SW1 SW_Push, SW2 SW_Push, SW3 SW_Push, SW4 SW_Push, SW5 SW_Push, SW6 SW_Push, SW7 RotaryEncoder_Switch, U1 MOUDLE-SEEEDUINO-XIAO

Commit message: ImtPad
Parts:
- moved U1 6.99 mm to (199.0, 76.0)
Changed lines of the file:
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@@
 	(footprint "Pretty:XIAO-Generic-Hybrid-14P-2.54-21X17.8MM"
 		(layer "B.Cu")
-		(at 192 76 90)
+		(at 198.99 76 90)
 		(property "Reference" "U1"
 			(at 0 -2.54 90)
@@
 	)
 	(segment
-		(start 197.08 68.375)
-		(end 197.08 62.08)
+		(start 204.07 68.375)
+		(end 204.07 62.08)
 		(width 0.2)
 		(layer "F.Cu")
@@
 	)
 	(segment
-		(start 193.39 79.935)
-		(end 193.39 60.54)
+		(start 200.38 79.935)
+		(end 200.38 60.54)
 		(width 0.2)
 		(layer "B.Cu")
@@
 	)
 	(segment
-		(start 197.08 83.625)
-		(end 193.39 79.935)
+		(start 204.07 83.625)
+		(end 200.38 79.935)
 		(width 0.2)
 		(layer "B.Cu")
@@
 	)
 	(segment
-		(start 186.92 83.625)
-		(end 176.955 73.66)
+		(start 193.91 83.625)
+		(end 183.945 73.66)
 		(width 0.2)
 		(layer "F.Cu")
@@
 	)
 	(segment
-		(start 199.62 86.38)
-		(end 199 87)
+		(start 206.61 86.38)
+		(end 205.99 87)
 		(width 0.2)
 		(layer "B.Cu")
@@
 	)
 	(segment
-		(start 199.62 83.625)
-		(end 199.62 86.38)
+		(start 206.61 83.625)
+		(end 206.61 86.38)
 		(width 0.2)
 		(layer "B.Cu")
@@
 	)
 	(segment
-		(start 199 87)
-		(end 122 87)
+		(start 205.99 87)
+		(end 128.99 87)
 		(width 0.2)
 		(layer "B.Cu")
@@
 	)
 	(segment
-		(start 188.36 82.525)
-		(end 132.897944 82.525)
+		(start 195.35 82.525)
+		(end 139.887944 82.525)
 		(width 0.2)
 		(layer "B.Cu")
@@
 	)
 	(segment
-		(start 189.46 83.625)
-		(end 188.36 82.525)
+		(start 196.45 83.625)
+		(end 195.35 82.525)
 		(width 0.2)
 		(layer "B.Cu")
@@
 	)
 	(segment
-		(start 192 83.625)
-		(end 190.375 82)
+		(start 198.99 83.625)
+		(end 197.365 82)
 		(width 0.2)
 		(layer "B.Cu")
@@
 	)
 	(segment
-		(start 190.375 82)
-		(end 135.826598 82)
+		(start 197.365 82)
+		(end 142.816598 82)
 		(width 0.2)
 		(layer "B.Cu")
@@
 	)
 	(segment
-		(start 194.54 83.625)
-		(end 167.64 56.725)
+		(start 201.53 83.625)
+		(end 174.63 56.725)
 		(width 0.2)
 		(layer "F.Cu")
@@
 	)
 	(segment
-		(start 186.92 68.375)
-		(end 186.92 55.92)
+		(start 193.91 68.375)
+		(end 193.91 55.92)
 		(width 0.2)
 		(layer "B.Cu")
@@
 	)
 	(segment
-		(start 184.38 68.375)
-		(end 184.38 59.13)
+		(start 191.37 68.375)
+		(end 191.37 59.13)
 		(width 0.2)
 		(layer "B.Cu")
@@
 	)
 	(segment
-		(start 191.01 69.925)
-		(end 199.696346 69.925)
+		(start 198 69.925)
+		(end 206.686346 69.925)
 		(width 0.2)
 		(layer "F.Cu")
@@
 	)
 	(segment
-		(start 199.696346 69.925)
-		(end 200.77 68.851346)
+		(start 206.686346 69.925)
+		(end 207.76 68.851346)
 		(width 0.2)
 		(layer "F.Cu")
@@
 	)
 	(segment
-		(start 189.46 68.375)
-		(end 191.01 69.925)
+		(start 196.45 68.375)
+		(end 198 69.925)
 		(width 0.2)
 		(layer "F.Cu")
@@
 	)
 	(segment
-		(start 200.77 68.851346)
-		(end 200.77 61.02)
+		(start 207.76 68.851346)
+		(end 207.76 61.02)
 		(width 0.2)
 		(layer "F.Cu")
