File: PCB/Imtpad.kicad_pcb (KiCad board)
At the start: 2 copper layers, 92 x 48 mm, 8 parts, among them SW1 SW_Push, SW2 SW_Push, SW3 SW_Push, SW4 SW_Push, SW5 SW_Push, SW6 SW_Push, SW7 RotaryEncoder_Switch, U1 MOUDLE-SEEEDUINO-XIAO

Commit message: ImtPad
Parts:
- moved U1 7.20 mm to (191.8, 76.0)
Routing:
- net Net-(U1-PA8_A4_D4_SDA): track 90.7 -> 33.7 mm
- net Net-(U1-PA02_A0_D0): track 119.2 -> 176.0 mm
- net Net-(U1-PA11_A3_D3): track 67.8 -> 10.9 mm
- net Net-(U1-PA4_A1_D1): track 75.1 -> 107.5 mm
- net unconnected-(U1-5V-Pad14): track 0.00 -> 24.6 mm
- net Net-(U1-PA5_A9_D9_MISO): track 25.2 -> 4.98 mm
- net GND: track 137.8 -> 151.9 mm
- net unconnected-(U1-3V3-Pad12): track 0.00 -> 12.5 mm
- net Net-(U1-PA7_A8_D8_SCK): track 18.0 -> 5.59 mm
- net unconnected-(U1-PA6_A10_D10_MOSI-Pad11): track 0.00 -> 9.24 mm
- net Net-(U1-PB09_A7_D7_RX): track 11.6 -> 2.31 mm
Other:
- board text added: "ImtPad V1"
Changed lines of the file:
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@@
 			(drillshape 0)
 			(scaleselection 1)
-			(outputdirectory "")
+			(outputdirectory "/home/imtiaz/Documents/ImtPad/production/gerbers/")
 		)
 	)
@@
 	(footprint "Pretty:XIAO-Generic-Hybrid-14P-2.54-21X17.8MM"
 		(layer "B.Cu")
-		(at 198.99 76 90)
+		(at 191.787985 76 90)
 		(property "Reference" "U1"
 			(at 0 -2.54 90)
@@
 		(layer "Edge.Cuts")
 	)
+	(gr_text "ImtPad V1"
+		(at 197.5 90 0)
+		(layer "F.Cu")
+		(effects
+			(font
+				(size 1.5 1.5)
+				(thickness 0.3)
+				(bold yes)
+			)
+			(justify left bottom)
+		)
+	)
+	(segment
+		(start 204 62.15)
+		(end 204.07 62.08)
+		(width 0.2)
+		(layer "F.Cu")
+		(net "GND")
+	)
+	(segment
+		(start 198 69.925)
+		(end 206.686346 69.925)
+		(width 0.2)
+		(layer "F.Cu")
+		(net "GND")
+	)
 	(segment
 		(start 190 55)
@@
 	)
 	(segment
+		(start 206.686346 69.925)
+		(end 207.76 68.851346)
+		(width 0.2)
+		(layer "F.Cu")
+		(net "GND")
+	)
+	(segment
+		(start 196.45 68.375)
+		(end 198 69.925)
+		(width 0.2)
+		(layer "F.Cu")
+		(net "GND")
+	)
+	(segment
+		(start 204.07 68.375)
+		(end 204 68.305)
+		(width 0.2)
+		(layer "F.Cu")
+		(net "GND")
+	)
+	(segment
 		(start 197.08 62.08)
 		(end 190 55)
@@
 	)
 	(segment
-		(start 197.25 52.5)
-		(end 194.75 55)
+		(start 207.76 68.851346)
+		(end 207.76 61.02)
 		(width 0.2)
 		(layer "F.Cu")
@@
 	)
 	(segment
-		(start 194.75 55)
-		(end 190 55)
+		(start 197.25 52.5)
+		(end 194.75 55)
 		(width 0.2)
 		(layer "F.Cu")
@@
 	)
 	(segment
-		(start 204.07 68.375)
-		(end 204.07 62.08)
+		(start 194.75 55)
+		(end 190 55)
 		(width 0.2)
 		(layer "F.Cu")
@@
 	)
 	(segment
-		(start 161.717056 54.61)
-		(end 148.59 54.61)
+		(start 195.35 82.525)
+		(end 139.887944 82.525)
 		(width 0.2)
 		(layer "B.Cu")
@@
 	)
 	(segment
-		(start 183.52 50.67)
-		(end 165.657056 50.67)
+		(start 161.717056 54.61)
+		(end 148.59 54.61)
 		(width 0.2)
 		(layer "B.Cu")
@@
 	)
 	(segment
-		(start 200.38 79.935)
-		(end 200.38 60.54)
+		(start 183.52 50.67)
+		(end 165.657056 50.67)
 		(width 0.2)
 		(layer "B.Cu")
@@
 	)
 	(segment
-		(start 204.07 83.625)
-		(end 200.38 79.935)
+		(start 196.45 83.625)
+		(end 195.35 82.525)
 		(width 0.2)
 		(layer "B.Cu")
@@
 	)
 	(segment
-		(start 193.91 83.625)
-		(end 183.945 73.66)
+		(start 186.92 83.625)
+		(end 176.955 73.66)
 		(width 0.2)
 		(layer "F.Cu")
@@
 	)
 	(segment
+		(start 198.99 83.625)
+		(end 197.365 82)
+		(width 0.2)
+		(layer "B.Cu")
+		(net "Net-(U1-PA02_A0_D0)")
+	)
+	(segment
 		(start 206.61 86.38)
 		(end 205.99 87)
@@
 	)
 	(segment
-		(start 205.99 87)
-		(end 128.99 87)
+		(start 197.365 82)
+		(end 142.816598 82)
 		(width 0.2)
 		(layer "B.Cu")
@@
 	)
 	(segment
-		(start 132.733402 72.26)
-		(end 134.133402 73.66)
+		(start 205.99 87)
+		(end 128.99 87)
 		(width 0.2)
 		(layer "B.Cu")
-		(net "Net-(U1-PA8_A4_D4_SDA)")
+		(net "Net-(U1-PA02_A0_D0)")
 	)
 	(segment
-		(start 195.35 82.525)
-		(end 139.887944 82.525)
+		(start 132.733402 72.26)
+		(end 134.133402 73.66)
 		(width 0.2)
 		(layer "B.Cu")
@@
 	)
 	(segment
-		(start 196.45 83.625)
-		(end 195.35 82.525)
-		(width 0.2)
-		(layer "B.Cu")
-		(net "Net-(U1-PA8_A4_D4_SDA)")
-	)
-	(segment
 		(start 127.07 74.150101)
 		(end 128.960101 72.26)
@@
 	)
 	(segment
-		(start 198.99 83.625)
-		(end 197.365 82)
-		(width 0.2)
-		(layer "B.Cu")
-		(net "Net-(U1-PA11_A3_D3)")
-	)
-	(segment
 		(start 135.826598 82)
 		(end 129.54 75.713402)
@@
 	)
 	(segment
-		(start 197.365 82)
-		(end 142.816598 82)
-		(width 0.2)
-		(layer "B.Cu")
-		(net "Net-(U1-PA11_A3_D3)")
-	)
-	(segment
 		(start 129.54 75.713402)
 		(end 129.54 73.66)
@@
 	)
 	(segment
-		(start 193.91 68.375)
-		(end 193.91 55.92)
-		(width 0.2)
-		(layer "B.Cu")
-		(net "Net-(U1-PA7_A8_D8_SCK)")
-	)
-	(segment
 		(start 183.5 52.5)
 		(end 182.75 52.5)
@@
 	)
 	(segment
-		(start 191.37 68.375)
-		(end 191.37 59.13)
-		(width 0.2)
-		(layer "B.Cu")
-		(net "Net-(U1-PB09_A7_D7_RX)")
-	)
-	(segment
 		(start 184.38 59.13)
 		(end 182.75 57.5)
@@
 	)
 	(segment
-		(start 198 69.925)
-		(end 206.686346 69.925)
+		(start 200.77 61.02)
+		(end 197.25 57.5)
 		(width 0.2)
 		(layer "F.Cu")
@@
 	)
 	(segment
-		(start 200.77 61.02)
-		(end 197.25 57.5)
+		(start 191.37 68.375)
+		(end 191.37 59.13)
 		(width 0.2)
-		(layer "F.Cu")
-		(net "Net-(U1-PA5_A9_D9_MISO)")
+		(layer "B.Cu")
+		(net "unconnected-(U1-PA6_A10_D10_MOSI-Pad11)")
 	)
 	(segment
-		(start 206.686346 69.925)
-		(end 207.76 68.851346)
+		(start 193.91 68.375)
+		(end 193.91 55.92)
 		(width 0.2)
-		(layer "F.Cu")
-		(net "Net-(U1-PA5_A9_D9_MISO)")
+		(layer "B.Cu")
+		(net "unconnected-(U1-3V3-Pad12)")
 	)
 	(segment
-		(start 196.45 68.375)
-		(end 198 69.925)
+		(start 200.38 79.935)
+		(end 200.38 60.54)
 		(width 0.2)
-		(layer "F.Cu")
-		(net "Net-(U1-PA5_A9_D9_MISO)")
+		(layer "B.Cu")
+		(net "unconnected-(U1-5V-Pad14)")
 	)
 	(segment
-		(start 207.76 68.851346)
-		(end 207.76 61.02)
+		(start 204.07 83.625)
+		(end 200.38 79.935)
 		(width 0.2)
-		(layer "F.Cu")
-		(net "Net-(U1-PA5_A9_D9_MISO)")
+		(layer "B.Cu")
+		(net "unconnected-(U1-5V-Pad14)")
 	)
 	(embedded_fonts no)
